File: TSAL.kicad_pcb (KiCad board)
At the start: 2 copper layers, 140 x 70 mm, 79 parts, among them J1 Mini-SPOX, J2 Mini-SPOX, J3 Mini-Fit_Jr, J4 Mini-SPOX, J5 Mini-SPOX, J6 Jumper, J7 Jumper, Q1 IRLML2502, Q2 IRLML2502, Q3 IRLML2502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

Commit message: changes
Parts:
- removed D5: FSV1045V, project:TO-277A_HandSolder
- added Q6: DMG3404L, Package_TO_SOT_SMD:SOT-23_Handsoldering, F.Cu at (168.0, 52.0)
- D1: value DFLS130L -> SMF4L15A
- R10: value 22k -> 130k
- R9: value 130k -> 22k
- moved C11 9.18 mm to (148.0, 66.0), turned to 270 degrees
- moved C12 6.80 mm to (140.5, 56.0)
- moved C10 5.39 mm to (138.0, 56.0)
- moved R10 5.39 mm to (145.0, 67.0), turned to 0 degrees
- moved R9 5.39 mm to (145.0, 65.0), turned to 180 degrees
- moved L1 5.00 mm to (155.0, 52.0)
- moved R13 5.00 mm to (137.0, 65.0)
- moved R14 5.00 mm to (137.0, 67.0)
- moved R8 5.00 mm to (140.0, 66.0)
- moved U5 5.00 mm to (143.0, 61.0)
- moved D1 4.72 mm to (133.0, 63.5), turned to 270 degrees
- moved C14 4.00 mm to (164.0, 57.0)
- moved D2 3.00 mm to (153.0, 63.0)
- moved G*** 2.24 mm to (151.0, 76.0)
- moved C9 0.50 mm to (129.0, 46.0)
Connections:
- C10 pad 1: Net-(C10-Pad1) -> /Power/VIN_F
- J7 pad 1: Net-(C14-Pad1) -> Net-(J7-Pad1)
- JP1 pad 1: Net-(C14-Pad1) -> Net-(J7-Pad1)
- R10 pad 1: Net-(R10-Pad1) -> Net-(C14-Pad1)
- R10 pad 2: GND -> Net-(R10-Pad2)
- R9 pad 1: Net-(C14-Pad1) -> Net-(R10-Pad2)
- R9 pad 2: Net-(R10-Pad1) -> GND
- U5 pad 2: Net-(C10-Pad1) -> /Power/VIN_F
- U5 pad 5: Net-(R10-Pad1) -> Net-(R10-Pad2)
Routing:
- net /Power/VIN_F: track 171.1 -> 214.4 mm, vias 2 -> 3
- net Net-(C12-Pad2): track 0.00 -> 7.42 mm, vias 4 -> 6
- net Net-(R10-Pad2): track 0.00 -> 4.31 mm
- net Net-(R10-Pad1): track 4.31 -> 0.00 mm
- net Net-(C12-Pad1): track 6.01 -> 2.12 mm, vias 2 -> 0
- net Net-(C11-Pad1): track 8.60 -> 5.96 mm, vias 2 -> 0
- net GND: track 61.0 -> 58.6 mm
- net Net-(C14-Pad1): track 31.4 -> 30.7 mm
- added copper zone on F.Cu, net Net-(J7-Pad1)
- removed copper zone on F.Cu, net Net-(C10-Pad1)
Other:
- board text added: "LEDs"
- board text added: "Power In"
- board text added: "Status Out"
- board text added: "TS Sense 1"
- board text added: "TS Sense 2"

Commit message: change to ideal diode controller
Parts:
- removed D4: DFLS130L, project:D_SOD-123_HandSolder
- removed Q6: DMG3404L, Package_TO_SOT_SMD:SOT-23_Handsoldering
- added TP5: TP_Vcap, TestPoint:TestPoint_Pad_D2.0mm, F.Cu at (234.0, 54.0)
- added TP6: TP_Vmid, TestPoint:TestPoint_Pad_D2.0mm, F.Cu at (234.0, 59.0)
- added TP7: TP_GND, TestPoint:TestPoint_Pad_D2.0mm, F.Cu at (234.0, 64.0)
- added U8: MAX40200AUK, Package_TO_SOT_SMD:SOT-23-5_HandSoldering, F.Cu at (235.0, 92.0)
- C16, C17, C18, C19: value 25 -> 35
- D3: value DFLS130L -> S1A; footprint project:D_SOD-123_HandSolder -> Diode_SMD:D_SMA_Handsoldering
- JP1: value Jumper_2_Bridged -> Jumper
- Q5: value IRLML6401 -> IRF8721; footprint Package_TO_SOT_SMD:SOT-23_Handsoldering -> Package_SO:SOIC-8_3.9x4.9mm_P1.27mm
- R4: value 22k -> 1k
- moved Q5 78.0 mm to (168.0, 53.0), turned to 0 degrees
- moved C9 15.7 mm to (115.0, 53.0), turned to 270 degrees
- moved C14 3.00 mm to (164.0, 60.0)
- moved D3 1.41 mm to (231.0, 91.0)
- moved C11 1.00 mm to (149.0, 66.0)
- moved R10 1.00 mm to (146.0, 67.0)
- moved R9 1.00 mm to (146.0, 65.0)
Connections:
- Q5 pad 1: Net-(C15-Pad1) -> Net-(C14-Pad1)
- Q5 pad 2: VCC -> Net-(C14-Pad1)
- Q5 pad 3: /Power/Vcap -> Net-(C14-Pad1)
Routing:
- net /Power/VIN_F: track 214.4 -> 225.6 mm
- net Net-(C16-Pad2): track 0.00 -> 11.0 mm
- net Net-(C15-Pad1): track 27.8 -> 20.1 mm
- net /Power/Vcap: track 203.9 -> 207.6 mm
- net VCC: track 232.5 -> 236.0 mm
- net Net-(L2-Pad1): track 6.48 -> 7.77 mm
- net Net-(C11-Pad1): track 5.96 -> 7.07 mm
- net Net-(R10-Pad2): track 4.31 -> 5.22 mm
- net GND: track 58.6 -> 59.5 mm, vias 22 -> 27
- net Net-(C14-Pad1): track 30.7 -> 30.2 mm

Commit message: last minute changes to test points and routing
Parts:
- TP1, TP2, TP3, TP4, TP5, TP6, TP7: footprint TestPoint:TestPoint_Pad_D2.0mm -> TestPoint:TestPoint_THTPad_D2.0mm_Drill1.0mm
- moved TP4 2.50 mm to (195.0, 100.0)
- moved TP2 2.00 mm to (187.0, 90.0)
- moved TP3 1.41 mm to (225.0, 99.0)
Routing:
- net Net-(C14-Pad1): track 30.2 -> 26.4 mm
- net +2V5: track 27.2 -> 29.7 mm
- net Net-(Q4-Pad1): track 36.0 -> 38.0 mm
- net VCC: track 236.0 -> 237.4 mm
- net Net-(C12-Pad2): vias 6 -> 2
- removed copper zone on B.Cu, net Net-(C12-Pad2)
