File: TSAL_Power.sch (KiCad schematic (older format))
At the start: 39 parts, among them J6 Jumper, J7 Jumper, Q5 IRLML6401, U5 LMR14030, U6 ZLDO1117G50, U7 TPS62205

Commit message: changes
Parts:
- removed D1: DFLS130L, project:D_SOD-123_HandSolder, symbol Device:D_Schottky
- removed D5: FSV1045V, project:TO-277A_HandSolder, symbol Device:D_Schottky_AAK
- added D1: SMF4L15A, project:D_SOD-123_HandSolder, symbol Device:D_Zener
- added Q6: DMG3404L, Package_TO_SOT_SMD:SOT-23_Handsoldering, symbol Device:Q_NMOS_GSD
- C10, C13, C14, C15, C22, C23: Part CL21A106KAYNNNE -> GRM21BC81E106KE11
- R13, R14: symbol Device:R -> Device:R_Small
- renumbered R9 to R10, R10 to R9
Connections:
- wire segments 73 -> 77
Other:
- note added: "UVLO 10V"
- note removed: "Lockout until\nVin > 10V"
- note removed: "reverse\npolarity\nprotection"
- moved on the sheet: C10, C11, C12, C14, C9, D2, F2, L1, R10, R13, R14, R8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

Commit message: change to ideal diode controller
Parts:
- removed D4: DFLS130L, project:D_SOD-123_HandSolder, symbol Device:D_Schottky
- removed Q5: IRLML6401, Package_TO_SOT_SMD:SOT-23_Handsoldering, symbol Device:Q_PMOS_GSD
- removed Q6: DMG3404L, Package_TO_SOT_SMD:SOT-23_Handsoldering, symbol Device:Q_NMOS_GSD
- added Q5: IRF8721, Package_SO:SOIC-8_3.9x4.9mm_P1.27mm, symbol Transistor_FET:IRF8721PBF-1
- added TP5: TP_Vcap, TestPoint:TestPoint_Pad_D2.0mm, symbol Connector:TestPoint
- added TP6: TP_Vmid, TestPoint:TestPoint_Pad_D2.0mm, symbol Connector:TestPoint
- added TP7: TP_GND, TestPoint:TestPoint_Pad_D2.0mm, symbol Connector:TestPoint
- added U8: MAX40200AUK, Package_TO_SOT_SMD:SOT-23-5_HandSoldering, symbol Analog_Switch:MAX40200AUK
- C16, C17, C18, C19: value 25 -> 35; Part SCCU25B256SRB -> SCCU30B356SRB
- D3: value DFLS130L -> S1A; footprint project:D_SOD-123_HandSolder -> Diode_SMD:D_SMA_Handsoldering; symbol Device:D_Schottky -> Device:D; Part DFLS130L-7 -> S1A
- JP1: value Jumper_2_Bridged -> Jumper; symbol Jumper:Jumper_2_Bridged -> Jumper:SolderJumper_2_Bridged
Connections:
- net GND: now also TP7.1, U8.2 (GND)
- net VCC: now also U8.5 (OUT)
- net VIN_F: now also Q5.4 (G)
- net Vcap: now also TP5.1, U8.1 (VDD), U8.3 (EN)
- net at C16.2, C17.1, C18.2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: now also TP6.1
- net at C14.1, L1.2, R10.1: now also Q5.1 (S), Q5.2 (S), Q5.3 (S)
- net at J7.1 (Pin_1), JP1.1 (A): now also Q5.5 (D), Q5.6 (D), Q5.7 (D), Q5.8 (D)
Other:
- note added: "SCCU30B356SRB"
- note removed: "SCCU25B256SRB"
- moved on the sheet: D3

Commit message: last minute changes to test points and routing
Parts:
- TP3, TP4, TP5, TP6, TP7: footprint TestPoint:TestPoint_Pad_D2.0mm -> TestPoint:TestPoint_THTPad_D2.0mm_Drill1.0mm
Changed lines of the file:
@@
 F 0 "TP4" H 10458 3018 50  0000 L CNN
 F 1 "TP_2V5" H 10458 2927 50  0000 L CNN
-F 2 "TestPoint:TestPoint_Pad_D2.0mm" H 10600 2900 50  0001 C CNN
+F 2 "TestPoint:TestPoint_THTPad_D2.0mm_Drill1.0mm" H 10600 2900 50  0001 C CNN
 F 3 "~" H 10600 2900 50  0001 C CNN
 	1    10400 2900
@@
 F 0 "TP3" H 10458 2018 50  0000 L CNN
 F 1 "TP_VCC" H 10458 1927 50  0000 L CNN
-F 2 "TestPoint:TestPoint_Pad_D2.0mm" H 10600 1900 50  0001 C CNN
+F 2 "TestPoint:TestPoint_THTPad_D2.0mm_Drill1.0mm" H 10600 1900 50  0001 C CNN
 F 3 "~" H 10600 1900 50  0001 C CNN
 	1    10400 1900
@@
 F 0 "TP5" V 6595 5072 50  0000 C CNN
 F 1 "TP_Vcap" V 6504 5072 50  0000 C CNN
-F 2 "TestPoint:TestPoint_Pad_D2.0mm" H 6600 5000 50  0001 C CNN
+F 2 "TestPoint:TestPoint_THTPad_D2.0mm_Drill1.0mm" H 6600 5000 50  0001 C CNN
 F 3 "~" H 6600 5000 50  0001 C CNN
 	1    6400 5000
@@
 F 0 "TP6" V 6595 5372 50  0000 C CNN
 F 1 "TP_Vmid" V 6504 5372 50  0000 C CNN
-F 2 "TestPoint:TestPoint_Pad_D2.0mm" H 6600 5300 50  0001 C CNN
+F 2 "TestPoint:TestPoint_THTPad_D2.0mm_Drill1.0mm" H 6600 5300 50  0001 C CNN
 F 3 "~" H 6600 5300 50  0001 C CNN
 	1    6400 5300
@@
 F 0 "TP7" V 6595 5672 50  0000 C CNN
 F 1 "TP_GND" V 6504 5672 50  0000 C CNN
-F 2 "TestPoint:TestPoint_Pad_D2.0mm" H 6600 5600 50  0001 C CNN
+F 2 "TestPoint:TestPoint_THTPad_D2.0mm_Drill1.0mm" H 6600 5600 50  0001 C CNN
 F 3 "~" H 6600 5600 50  0001 C CNN
 	1    6400 5600
