File: TSAL_LED.kicad_pcb (KiCad board)
At the start: 2 copper layers, 104.1 x 45.8 mm, 70 parts, among them J1 Mini-SPOX, U1 XC9141, U2 XC9141

Commit message: remove boost converter for RLED
Parts:
- removed L1: 4.7uH, Inductor_SMD:L_Coilcraft_LPS5030
- removed U1: XC9141, Package_TO_SOT_SMD:SOT-23-5_HandSoldering
- added D21: D, project:d0214ba, F.Cu at (128.9, 78.1)
- added Q1: Q_PMOS_GSD, Package_TO_SOT_SMD:SOT-23, F.Cu at (137.8, 81.9)
- added TP1: TestPoint, TestPoint:TestPoint_Pad_D3.0mm, F.Cu at (128.9, 82.5)
Connections:
- U2 pad 4: /LED+ -> Net-(D21-Pad2)
Routing:
- net +2V5: track 56.3 -> 47.4 mm
- net Net-(D21-Pad2): track 0.00 -> 8.03 mm
- net Net-(L1-Pad2): track 6.25 -> 0.00 mm
- net /RLED-: track 234.5 -> 232.3 mm
- net /LED+: track 231.9 -> 232.7 mm

Commit message: shuffled some files around, generated gerbers
Parts:
- removed D21: D, project:d0214ba
Connections:
- Q1 pad 2: /LED+ -> +2V5
- Q1 pad 3: +2V5 -> /LED+
- TP1 pad 1: Net-(D21-Pad2) -> /LED+
- U2 pad 4: Net-(D21-Pad2) -> /LED+
Routing:
- net Net-(D21-Pad2): track 8.03 -> 0.00 mm
- net /LED+: track 232.7 -> 240.5 mm
- net +2V5: track 47.4 -> 48.1 mm
Changed lines of the file:
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@@
     (thickness 1.6)
     (drawings 14)
-    (tracks 376)
+    (tracks 374)
     (zones 0)
-    (modules 71)
-    (nets 67)
+    (modules 70)
+    (nets 66)
   )
   (page A4)
@@
   )
   (setup
-    (last_trace_width 0.5)
+    (last_trace_width 0.25)
     (user_trace_width 0.5)
     (trace_clearance 0.2)
@@
       (outputformat 1)
       (mirror false)
-      (drillshape 1)
+      (drillshape 0)
       (scaleselection 1)
-      (outputdirectory ""))
+      (outputdirectory "gerber/TSAL_LED/"))
   )
   (net 0 "")
@@
   (net 64 /LED+)
   (net 65 "Net-(L2-Pad2)")
-  (net 66 "Net-(D21-Pad2)")
   (net_class Default "This is the default net class."
     (clearance 0.2)
@@
     (add_net "Net-(D20-Pad3)")
     (add_net "Net-(D20-Pad4)")
-    (add_net "Net-(D21-Pad2)")
     (add_net "Net-(D3-Pad1)")
     (add_net "Net-(D3-Pad3)")
@@
     (tags "test point SMD pad")
     (attr virtual)
-    (fp_text reference TP1 (at 0 -2.398) (layer F.SilkS)
+    (fp_text reference TP1 (at 3.175 0 90) (layer F.SilkS)
       (effects (font (size 1 1) (thickness 0.15)))
     )
@@
     )
     (pad 1 smd circle (at 0 0) (size 3 3) (layers F.Cu F.Mask)
-      (net 66 "Net-(D21-Pad2)"))
+      (net 64 /LED+))
   )
   (module Package_TO_SOT_SMD:SOT-23 (layer F.Cu)
@@
     )
     (pad 3 smd rect (at 1 0 270) (size 0.9 0.8) (layers F.Cu F.Paste F.Mask)
-      (net 3 +2V5))
-    (pad 2 smd rect (at -1 0.95 270) (size 0.9 0.8) (layers F.Cu F.Paste F.Mask)
       (net 64 /LED+))
+    (pad 2 smd rect (at -1 0.95 270) (size 0.9 0.8) (layers F.Cu F.Paste F.Mask)
+      (net 3 +2V5))
     (pad 1 smd rect (at -1 -0.95 270) (size 0.9 0.8) (layers F.Cu F.Paste F.Mask)
       (net 63 /RLED-))
@@
     )
   )
-  (module project:d0214ba (layer F.Cu)
-    (at 128.94 78.105 180)
-    (descr "Microsemi LSM115J")
-    (tags "DO-214BA diode")
-    (attr smd)
-    (fp_text reference D21 (at -3.5 0 90) (layer F.SilkS)
-      (effects (font (size 1.016 1.016) (thickness 0.254)))
-    )
-    (fp_text value D (at 0 3) (layer F.SilkS) hide
-      (effects (font (size 1 1) (thickness 0.15)))
-    )
-    (fp_line (start 2.25 1.95) (end -2.25 1.95) (layer F.SilkS) (width 0.15))
-    (fp_line (start -2.25 -1.95) (end 2.25 -1.95) (layer F.SilkS) (width 0.15))
-    (fp_line (start -1.2 -1.55) (end -1.2 -1.95) (layer F.SilkS) (width 0.15))
-    (fp_line (start -1.35 -1.55) (end -1.2 -1.55) (layer F.SilkS) (width 0.15))
-    (fp_line (start -1.35 -1.95) (end -1.35 -1.55) (layer F.SilkS) (width 0.15))
-    (fp_line (start -1.2 1.55) (end -1.2 1.95) (layer F.SilkS) (width 0.15))
-    (fp_line (start -1.35 1.55) (end -1.2 1.55) (layer F.SilkS) (width 0.15))
-    (fp_line (start -1.35 1.95) (end -1.35 1.55) (layer F.SilkS) (width 0.15))
-    (fp_line (start 2.25 -1.95) (end 2.25 -1.55) (layer F.SilkS) (width 0.15))
-    (fp_line (start 2.25 1.95) (end 2.25 1.55) (layer F.SilkS) (width 0.15))
-    (fp_line (start -2.25 1.95) (end -2.25 1.55) (layer F.SilkS) (width 0.15))
-    (fp_line (start -2.25 -1.95) (end -2.25 -1.55) (layer F.SilkS) (width 0.15))
-    (fp_line (start -3 2.25) (end -3 -2.25) (layer F.CrtYd) (width 0.05))
-    (fp_line (start 3 2.25) (end -3 2.25) (layer F.CrtYd) (width 0.05))
-    (fp_line (start 3 -2.25) (end 3 2.25) (layer F.CrtYd) (width 0.05))
-    (fp_line (start -3 -2.25) (end 3 -2.25) (layer F.CrtYd) (width 0.05))
-    (pad 1 smd rect (at -1.94 0 180) (size 2.71 2.5) (layers F.Cu F.Paste F.Mask)
-      (net 64 /LED+))
-    (pad 2 smd rect (at 1.94 0 180) (size 2.71 2.5) (layers F.Cu F.Paste F.Mask)
-      (net 66 "Net-(D21-Pad2)"))
-  )
   (module project:OUR-Logo (layer B.Cu)
     (at 125.095 76.835 180)
@@
       (net 65 "Net-(L2-Pad2)"))
     (pad 4 smd rect (at 1.35 0.95 90) (size 1.56 0.65) (layers F.Cu F.Paste F.Mask)
-      (net 66 "Net-(D21-Pad2)"))
+      (net 64 /LED+))
     (pad 3 smd rect (at -1.35 0.95 90) (size 1.56 0.65) (layers F.Cu F.Paste F.Mask)
       (net 3 +2V5))
@@
   (segment (start 124.46 83.83) (end 125.72 85.09) (width 0.5) (layer F.Cu) (net 3))
   (segment (start 124.46 82.55) (end 124.46 83.83) (width 0.5) (layer F.Cu) (net 3))
-  (segment (start 125.72 85.09) (end 141.605 85.09) (width 0.5) (layer F.Cu) (net 3))
   (segment (start 147.4 85.165) (end 147.4 85.09) (width 0.5) (layer F.Cu) (net 3))
   (segment (start 148.75 86.515) (end 147.4 85.165) (width 0.5) (layer F.Cu) (net 3))
@@
   (segment (start 147.4 85.09) (end 147.4 85.015) (width 0.5) (layer F.Cu) (net 3))
   (segment (start 140.87 85.09) (end 141.605 85.09) (width 0.5) (layer F.Cu) (net 3))
-  (segment (start 138.695 82.915) (end 140.87 85.09) (width 0.5) (layer F.Cu) (net 3))
-  (segment (start 137.795 82.915) (end 138.695 82.915) (width 0.5) (layer F.Cu) (net 3))
+  (segment (start 136.845 80.915) (end 136.845 80.965) (width 0.5) (layer F.Cu) (net 3))
+  (segment (start 136.845 80.915) (end 136.845 84.14) (width 0.5) (layer F.Cu) (net 3))
+  (segment (start 136.845 84.14) (end 137.795 85.09) (width 0.5) (layer F.Cu) (net 3))
+  (segment (start 125.72 85.09) (end 137.795 85.09) (width 0.5) (layer F.Cu) (net 3))
+  (segment (start 137.795 85.09) (end 141.605 85.09) (width 0.5) (layer F.Cu) (net 3))
   (segment (start 106.045 64.53) (end 106.045 59.055) (width 0.5) (layer F.Cu) (net 4))
   (segment (start 109.855 70.485) (end 109.855 75.96) (width 0.5) (layer F.Cu) (net 5))
@@
   (segment (start 139.54 77.71) (end 138.745 78.505) (width 0.5) (layer F.Cu) (net 63))
   (via (at 140.97 79.375) (size 0.8) (drill 0.4) (layers F.Cu B.Cu) (net 64))
-  (via (at 131.445 76.2) (size 0.8) (drill 0.4) (layers F.Cu B.Cu) (net 64))
+  (via (at 128.905 76.2) (size 0.8) (drill 0.4) (layers F.Cu B.Cu) (net 64))
   (segment (start 157.546985 65.324999) (end 162.820001 65.324999) (width 0.5) (layer B.Cu) (net 64))
   (segment (start 153.930001 60.244999) (end 154.58999 60.904988) (width 0.5) (layer B.Cu) (net 64))
@@
   (segment (start 145.415 74.93) (end 145.415 70.485) (width 0.5) (layer B.Cu) (net 64))
   (segment (start 140.97 79.375) (end 145.415 74.93) (width 0.5) (layer B.Cu) (net 64))
-  (segment (start 130.88 76.765) (end 131.445 76.2) (width 0.5) (layer F.Cu) (net 64))
-  (segment (start 130.88 78.105) (end 130.88 76.765) (width 0.5) (layer F.Cu) (net 64))
-  (segment (start 131.445 76.2) (end 130.175 74.93) (width 0.5) (layer B.Cu) (net 64))
-  (segment (start 140.97 79.940685) (end 140.97 79.375) (width 0.5) (layer F.Cu) (net 64))
-  (segment (start 139.455002 81.865) (end 140.97 80.350002) (width 0.5) (layer F.Cu) (net 64))
-  (segment (start 137.745 81.865) (end 139.455002 81.865) (width 0.5) (layer F.Cu) (net 64))
-  (segment (start 136.845 80.965) (end 137.745 81.865) (width 0.5) (layer F.Cu) (net 64))
-  (segment (start 140.97 80.350002) (end 140.97 79.940685) (width 0.5) (layer F.Cu) (net 64))
-  (segment (start 136.845 80.915) (end 136.845 80.965) (width 0.5) (layer F.Cu) (net 64))
+  (segment (start 138.695 82.915) (end 137.795 82.915) (width 0.5) (layer F.Cu) (net 64))
+  (segment (start 140.97 80.64) (end 138.695 82.915) (width 0.5) (layer F.Cu) (net 64))
+  (segment (start 140.97 79.375) (end 140.97 80.64) (width 0.5) (layer F.Cu) (net 64))
+  (segment (start 125.255 79.85) (end 127 78.105) (width 0.5) (layer F.Cu) (net 64))
+  (segment (start 124.46 79.85) (end 125.255 79.85) (width 0.5) (layer F.Cu) (net 64))
+  (segment (start 127.405001 81.050001) (end 126.455001 81.050001) (width 0.5) (layer F.Cu) (net 64))
+  (segment (start 126.455001 81.050001) (end 125.255 79.85) (width 0.5) (layer F.Cu) (net 64))
+  (segment (start 128.905 82.55) (end 127.405001 81.050001) (width 0.5) (layer F.Cu) (net 64))
+  (segment (start 127 78.105) (end 128.905 76.2) (width 0.5) (layer F.Cu) (net 64))
+  (segment (start 128.905 76.2) (end 130.175 74.93) (width 0.5) (layer B.Cu) (net 64))
   (segment (start 117.95 79.85) (end 116.84 78.74) (width 0.5) (layer F.Cu) (net 65))
   (segment (start 122.56 79.85) (end 117.95 79.85) (width 0.5) (layer F.Cu) (net 65))
-  (segment (start 125.255 79.85) (end 127 78.105) (width 0.5) (layer F.Cu) (net 66))
-  (segment (start 124.46 79.85) (end 125.255 79.85) (width 0.5) (layer F.Cu) (net 66))
-  (segment (start 127.405001 81.050001) (end 126.455001 81.050001) (width 0.5) (layer F.Cu) (net 66))
-  (segment (start 126.455001 81.050001) (end 125.255 79.85) (width 0.5) (layer F.Cu) (net 66))
-  (segment (start 128.905 82.55) (end 127.405001 81.050001) (width 0.5) (layer F.Cu) (net 66))
 )
