File: TSAL.sch (KiCad schematic (older format))
At the start: 39 parts, among them J1 Mini-SPOX, J2 Mini-SPOX, J3 Mini-Fit_Jr, J4 Mini-SPOX, J5 Mini-SPOX, Q1 IRLML2502, Q2 IRLML2502, Q3 IRLML2502, Q4 IRLML2502, U1 74HC08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

Commit message: changes
Parts:
- C1, C4: Part CL21A106KAYNNNE -> GRM21BC81E106KE11
Changed lines of the file:
@@
 F 2 "Capacitor_SMD:C_0805_2012Metric_Pad1.15x1.40mm_HandSolder" H 4738 6000 50  0001 C CNN
 F 3 "~" H 4700 6150 50  0001 C CNN
-F 4 "CL21A106KAYNNNE" H 4700 6150 50  0001 C CNN "Part"
+F 4 "GRM21BC81E106KE11" H 4700 6150 50  0001 C CNN "Part"
 	1    4700 6150
 	1    0    0    -1
@@
 F 2 "Capacitor_SMD:C_0805_2012Metric_Pad1.15x1.40mm_HandSolder" H 5838 6000 50  0001 C CNN
 F 3 "~" H 5800 6150 50  0001 C CNN
-F 4 "CL21A106KAYNNNE" H 5800 6150 50  0001 C CNN "Part"
+F 4 "GRM21BC81E106KE11" H 5800 6150 50  0001 C CNN "Part"
 	1    5800 6150
 	1    0    0    -1

Commit message: change to ideal diode controller
Parts:
- R4: value 22k -> 1k; Part RC0805FR-0722KL -> RC0805FR-071KL
Changed lines of the file:
@@
 P 5850 4800
 F 0 "R4" V 5643 4800 50  0000 C CNN
-F 1 "22k" V 5734 4800 50  0000 C CNN
+F 1 "1k" V 5734 4800 50  0000 C CNN
 F 2 "Resistor_SMD:R_0805_2012Metric_Pad1.15x1.40mm_HandSolder" V 5780 4800 50  0001 C CNN
 F 3 "~" H 5850 4800 50  0001 C CNN
-F 4 "RC0805FR-0722KL" H 5850 4800 50  0001 C CNN "Part"
+F 4 "RC0805FR-071KL" H 5850 4800 50  0001 C CNN "Part"
 	1    5850 4800
 	0    1    1    0

Commit message: last minute changes to test points and routing
Parts:
- TP1, TP2: footprint TestPoint:TestPoint_Pad_D2.0mm -> TestPoint:TestPoint_THTPad_D2.0mm_Drill1.0mm
Changed lines of the file:
@@
 F 0 "TP2" H 8258 3918 50  0000 L CNN
 F 1 "TP_RLED_Ctrl" H 8258 3827 50  0000 L CNN
-F 2 "TestPoint:TestPoint_Pad_D2.0mm" H 8400 3800 50  0001 C CNN
+F 2 "TestPoint:TestPoint_THTPad_D2.0mm_Drill1.0mm" H 8400 3800 50  0001 C CNN
 F 3 "~" H 8400 3800 50  0001 C CNN
 	1    8200 3800
@@
 F 0 "TP1" H 6158 3518 50  0000 L CNN
 F 1 "TP_Timer_En" H 6158 3427 50  0000 L CNN
-F 2 "TestPoint:TestPoint_Pad_D2.0mm" H 6300 3400 50  0001 C CNN
+F 2 "TestPoint:TestPoint_THTPad_D2.0mm_Drill1.0mm" H 6300 3400 50  0001 C CNN
 F 3 "~" H 6300 3400 50  0001 C CNN
 	1    6100 3400

Commit message: tsal sense board update
hopefully last update
Parts:
- U4: symbol Timer:LM555 -> Timer:LM555xM
Changed lines of the file:
@@
 	5000 5000 5000 6100
 $Comp
-L Timer:LM555 U4
+L Timer:LM555xM U4
 U 1 1 5DA76938
 P 7400 4300
