File: HV_Sense/TSAL_HV_Sense.sch (KiCad schematic (older format))
At the start: 26 parts, among them J1 Nano-Fit, J2 Mini-SPOX, J3 Nano-Fit, J4 Mini-SPOX, J5 Mini-SPOX, J6 Mini-SPOX, U1 4N35, U2 4N35

Commit message: HV_Sense: change hv input connector to Micro-Fit
Parts:
- J1, J3: value Nano-Fit -> Micro-Fit; footprint Connector_Molex:Molex_Nano-Fit_105309-xx02_1x02_P2.50mm_Vertical -> Connector_Molex:Molex_Micro-Fit_3.0_43650-0215_1x02_P3.00mm_Vertical; Part 105309-1102 -> 43650-0216
Changed lines of the file:
@@
 P 3500 4550
 F 0 "J3" H 3418 4317 50  0000 C CNN
-F 1 "Nano-Fit" H 3418 4316 50  0001 C CNN
-F 2 "Connector_Molex:Molex_Nano-Fit_105309-xx02_1x02_P2.50mm_Vertical" H 3500 4550 50  0001 C CNN
+F 1 "Micro-Fit" H 3418 4316 50  0001 C CNN
+F 2 "Connector_Molex:Molex_Micro-Fit_3.0_43650-0215_1x02_P3.00mm_Vertical" H 3500 4550 50  0001 C CNN
 F 3 "~" H 3500 4550 50  0001 C CNN
-F 4 "105309-1102" H 3500 4550 50  0001 C CNN "Part"
+F 4 "43650-0216" H 3500 4550 50  0001 C CNN "Part"
 	1    3500 4550
 	-1   0    0    1
@@
 P 4100 2550
 F 0 "J1" H 4018 2317 50  0000 C CNN
-F 1 "Nano-Fit" H 4018 2316 50  0001 C CNN
-F 2 "Connector_Molex:Molex_Nano-Fit_105309-xx02_1x02_P2.50mm_Vertical" H 4100 2550 50  0001 C CNN
+F 1 "Micro-Fit" H 4018 2316 50  0001 C CNN
+F 2 "Connector_Molex:Molex_Micro-Fit_3.0_43650-0215_1x02_P3.00mm_Vertical" H 4100 2550 50  0001 C CNN
 F 3 "~" H 4100 2550 50  0001 C CNN
-F 4 "105309-1102" H 4100 2550 50  0001 C CNN "Part"
+F 4 "43650-0216" H 4100 2550 50  0001 C CNN "Part"
 	1    4100 2550
 	-1   0    0    1

Commit message: HV_Sense: update schematics
Parts:
- R2: symbol Device:R -> Device:R_Small
Connections:
- net AUX_1: no longer names the net of J5.1 (Pin_1), J6.3 (Pin_3), R12.1, R9.2
- net AUX_2: no longer names the net of J5.2 (Pin_2), J6.2 (Pin_2), R11.1, R8.2
- net AUX_3: no longer names the net of J5.3 (Pin_3), J6.1 (Pin_1), R10.1, R7.2
- net GND: no longer names the net of J2.1 (Pin_1), U1.4
- net GND: no longer J6.5 (Pin_5), U2.4
- net HV+: no longer names the net of D2.1 (K), D3.1 (K), J3.2 (Pin_2)
- net HV+: no longer D1.1 (K), J1.2 (Pin_2)
- net HV-: no longer names the net of J3.1 (Pin_1), J4.1 (Pin_1), U2.2
- net HV-: no longer J1.1 (Pin_1), U1.2
- net Sense: no longer names the net of J2.2 (Pin_2), R2.2, U1.5
- net Sense: no longer J6.6 (Pin_6), R6.1, U2.5
- net VCC: no longer names the net of D4.2 (A), D5.2 (A), D6.2 (A), J6.4 (Pin_4), R6.2, R7.1, R8.1, R9.1
- net VCC: no longer J2.3 (Pin_3), R2.1
- new net: J2.3 (Pin_3), R2.1
- new net: J1.1 (Pin_1), U1.2
- new net: D1.1 (K), J1.2 (Pin_2)
- new net: J6.5 (Pin_5), U2.4
- new net: J6.6 (Pin_6), R6.1, U2.5
Other:
- note added: "AUX_1"
- note added: "AUX_2"
- note added: "AUX_3"
- note added: "GND"
- note added: "HV+"
- note added: "HV-"
- note added: "Sense"
- note added: "VCC"
- note removed: "To HVJB (TSAL Logic Board)"
- moved on the sheet: D2, D3, D4, D5, D6, J3, J4, J5, J6, R10, R11, R12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
