File: Main/TSAL_Power.sch (KiCad schematic (older format))
At the start: 41 parts, among them J6 Jumper, J7 Jumper, Q5 IRF8721, U5 LMR14030, U6 ZLDO1117G50, U7 TPS62205, U8 MAX40200AUK

Commit message: Main board: Rev B schematics design
major redesign of power delivery and backup
Parts:
- removed C10: 10u, Capacitor_SMD:C_0805_2012Metric_Pad1.15x1.40mm_HandSolder, symbol Device:C_Small
- removed C11, C12: 100n, Capacitor_SMD:C_0805_2012Metric_Pad1.15x1.40mm_HandSolder, symbol Device:C_Small
- removed C15: 10u, Capacitor_SMD:C_0805_2012Metric_Pad1.15x1.40mm_HandSolder, symbol Device:C
- removed C16, C17, C18, C19: 35, Capacitor_THT:CP_Radial_D16.0mm_P7.50mm, symbol Device:CP
- removed C20, C21: DNP, Capacitor_THT:CP_Radial_D16.0mm_P7.50mm, symbol Device:CP
- removed C9: 100u, Capacitor_THT:CP_Radial_D5.0mm_P2.50mm, symbol Device:CP1
- removed D2: FSV1045V, project:TO-277A_HandSolder, symbol project:D_Schottky_Small_AAK
- removed D3: S1A, Diode_SMD:D_SMA_Handsoldering, symbol Device:D
- removed J6, J7: Jumper, Connector_PinHeader_2.54mm:PinHeader_1x02_P2.54mm_Vertical, symbol Connector_Generic:Conn_01x02
- removed JP1: Jumper, Jumper:SolderJumper-2_P1.3mm_Open_Pad1.0x1.5mm, symbol Jumper:SolderJumper_2_Bridged
- removed Q5: IRF8721, Package_SO:SOIC-8_3.9x4.9mm_P1.27mm, symbol Transistor_FET:IRF8721PBF-1
- removed R10: 130k, Resistor_SMD:R_0805_2012Metric_Pad1.15x1.40mm_HandSolder, symbol Device:R
- removed R11: 1k, Resistor_SMD:R_0805_2012Metric_Pad1.15x1.40mm_HandSolder, symbol Device:R
- removed R8: 100k, Resistor_SMD:R_0805_2012Metric_Pad1.15x1.40mm_HandSolder, symbol Device:R
- removed R9: 22k, Resistor_SMD:R_0805_2012Metric_Pad1.15x1.40mm_HandSolder, symbol Device:R
- removed U5: LMR14030, Package_SO:SOIC-8-1EP_3.9x4.9mm_P1.27mm_EP2.41x3.3mm, symbol project:LMR140x0
- removed U6: ZLDO1117G50, Package_TO_SOT_SMD:SOT-223-3_TabPin2, symbol Regulator_Linear:AMS1117-5.0
- removed U7: TPS62205, Package_TO_SOT_SMD:SOT-23-5_HandSoldering, symbol Regulator_Switching:TPS62205DBV
- added C10, C11, C12, C9: 10uF, Capacitor_SMD:C_0805_2012Metric, symbol Device:C
- added C15, C16, C17, C20, C21, C25, C28, C29, C35, C38, C40, C41, C43, C6: 0.1uF, Capacitor_SMD:C_0402_1005Metric, symbol Device:C_Small
- added C18, C19: 220uF, Capacitor_SMD:CP_Elec_8x10.5, symbol Device:C_Polarized_US
- added C24, C7, C8: 10uF, Capacitor_SMD:C_1210_3225Metric, symbol Device:C
- added C26: 10uF, Capacitor_SMD:C_0805_2012Metric, symbol Device:C_Small
- added C27: 150pF, Capacitor_SMD:C_0402_1005Metric, symbol Device:C_Small
- added C30, C31, C32: 100uF, Capacitor_SMD:C_1210_3225Metric, symbol Device:C
- added C33, C34, C36, C37: 200F, Capacitor_THT:CP_Radial_D30.0mm_P10.00mm_SnapIn, symbol Device:C_Polarized_US
- added C39, C42, C44: 1nF, Capacitor_SMD:C_0402_1005Metric, symbol Device:C_Small
- added D1: ~, Diode_SMD:D_SOD-123, symbol Device:D
- added D3: ~, Diode_SMD:D_SOD-323, symbol Device:D_Schottky_Small_Filled
- added F2: 1A, Fuse:Fuseholder_Littelfuse_Nano2_154x, symbol Device:Fuse
- added JP1: 0, Resistor_SMD:R_0402_1005Metric, symbol Jumper:SolderJumper_2_Open
- added L3: 2.2uH, Inductor_SMD:L_Bourns-SRN8040_8x8.15mm, symbol Device:L
- added L4: 3.3uH, Inductor_SMD:L_Bourns_SRP1245A, symbol Device:L
- added Q10: NPN, Package_TO_SOT_SMD:SOT-23, symbol Device:Q_NPN_BEC
- added Q11, Q9: MJD122, Package_TO_SOT_SMD:TO-252-2, symbol Device:Q_NPN_Darlington_BCE
- added Q12: PNP, Package_TO_SOT_SMD:SOT-23, symbol Device:Q_PNP_BEC
- added Q6: BSC0904NSI, Package_TO_SOT_SMD:TDSON-8-1, symbol project:NMOS_SuperSO8
- added Q7, Q8: BSC0902NSI, Package_TO_SOT_SMD:TDSON-8-1, symbol project:NMOS_SuperSO8
- added R15, R30: 56k, Resistor_SMD:R_0805_2012Metric, symbol Device:R_Small
- added R16, R19, R48, R49: 10k, Resistor_SMD:R_0805_2012Metric, symbol Device:R_Small
- added R17, R28: 68k, Resistor_SMD:R_0805_2012Metric, symbol Device:R_Small
- added R18, R20, R21, R22, R23, R26, R29, R32, R35, R36, R41: 10k, Resistor_SMD:R_0402_1005Metric, symbol Device:R_Small
- added R24, R25: 0, Resistor_SMD:R_0402_1005Metric, symbol Device:R_Small
- added R27, R45, R50: 15k, Resistor_SMD:R_0805_2012Metric, symbol Device:R_Small
- added R31: 0.006, Resistor_SMD:R_2512_6332Metric, symbol Device:R
- added R33, R38, R44: 47k, Resistor_SMD:R_0805_2012Metric, symbol Device:R_Small
- added R34: 12k, Resistor_SMD:R_0805_2012Metric, symbol Device:R_Small
- added R37, R40, R42, R43, R47: 1k, Resistor_SMD:R_0402_1005Metric, symbol Device:R_Small
- added R39, R46: 100k, Resistor_SMD:R_0402_1005Metric, symbol Device:R_Small
- added TP1, TP10, TP11, TP12, TP2, TP8, TP9: ~, TestPoint:TestPoint_Loop_D2.50mm_Drill1.0mm, symbol Connector:TestPoint
- added U10, U11: TLV431, Package_TO_SOT_SMD:SOT-23, symbol Reference_Voltage:TL432DBZ
- added U4: TPS562200, Package_TO_SOT_SMD:SOT-23-6, symbol Regulator_Switching:TPS562200
- added U5: TPS63020, project:TPS63020, symbol project:TPS63020
- added U7: INA180A3, Package_TO_SOT_SMD:SOT-23-5, symbol project:INA180A
- added U8: TLV9104, Package_SO:TSSOP-14_4.4x5mm_P0.65mm, symbol Device:Opamp_Quad
- added U9: LM25117, Package_SO:ETSSOP-20-1EP_4.4x6.5mm_P0.65mm_EP3x4.2mm, symbol project:LM5117PMH
- added ZZ1, ZZ2, ZZ4, ZZ5, ZZ6, ZZ7, ZZ9: ~, project:Trace_0.2mmx0.6mm, symbol project:Wire
- added ZZ3: ~, project:Trace_1mmx2mm, symbol project:Wire
- added ZZ8: ~, project:Trace_0.4mmx0.8mm, symbol project:Wire
- C13, C14: value 10u -> 10uF; footprint Capacitor_SMD:C_0805_2012Metric_Pad1.15x1.40mm_HandSolder -> Capacitor_SMD:C_0805_2012Metric; Part GRM21BC81E106KE11 -> (none)
- C22, C23: value 10u -> 10uF; footprint Capacitor_SMD:C_0805_2012Metric_Pad1.15x1.40mm_HandSolder -> Capacitor_SMD:C_1210_3225Metric; Comment (none) -> 25V; Part GRM21BC81E106KE11 -> (none)
- D2: renamed from D1; footprint project:D_SOD-123_HandSolder -> Diode_SMD:D_SOD-123
- F1: renamed from F2; value 3A -> 6A; footprint Fuse:Fuseholder_Cylinder-5x20mm_Schurter_0031_8201_Horizontal_Open -> Fuse:Fuseholder_Littelfuse_Nano2_154x; Part 0031.8201 -> 15406.3
- L1: value 15u -> 1uH; footprint project:104CDMCCDS -> Inductor_SMD:L_1206_3216Metric; Part 104CDMCCDS-150MC -> LB3218T1R0M
- L2: value 10u -> 4.7uH; footprint project:CDRH62B -> Inductor_SMD:L_Bourns-SRN4018; Part CDRH62BNP-100MC-B -> SRN4018-4R7M
- R12: value 4.7 -> 0.006; footprint Resistor_THT:R_Axial_DIN0516_L15.5mm_D5.0mm_P20.32mm_Horizontal -> Resistor_SMD:R_2512_6332Metric; Part AC03000004708JAC00 -> LRMAP2512-R006
- R13: value 820k -> 56k; footprint Resistor_SMD:R_0805_2012Metric_Pad1.15x1.40mm_HandSolder -> Resistor_SMD:R_0805_2012Metric; Part RC0805FR-07820KL -> (none)
- R14: value 100k -> 10k; footprint Resistor_SMD:R_0805_2012Metric_Pad1.15x1.40mm_HandSolder -> Resistor_SMD:R_0805_2012Metric; Part RC0805FR-07100KL -> (none)
- TP3: value TP_VCC -> ~; footprint TestPoint:TestPoint_THTPad_D2.0mm_Drill1.0mm -> TestPoint:TestPoint_Loop_D2.50mm_Drill1.0mm; Comment (none) -> 5V; DNP (none) -> DNP; Part (none) -> Keystone 5000
- TP4: value TP_2V5 -> ~; footprint TestPoint:TestPoint_THTPad_D2.0mm_Drill1.0mm -> TestPoint:TestPoint_Loop_D2.50mm_Drill1.0mm; Comment (none) -> VCC; DNP (none) -> DNP; Part (none) -> Keystone 5000
- TP5: value TP_Vcap -> ~; footprint TestPoint:TestPoint_THTPad_D2.0mm_Drill1.0mm -> TestPoint:TestPoint_Loop_D2.50mm_Drill1.0mm; Comment (none) -> GND; DNP (none) -> DNP; Part (none) -> Keystone 5000
- TP6: value TP_Vmid -> ~; footprint TestPoint:TestPoint_THTPad_D2.0mm_Drill1.0mm -> TestPoint:TestPoint_Loop_D2.50mm_Drill1.0mm; Comment (none) -> I_IN; DNP (none) -> DNP; Part (none) -> Keystone 5000
- TP7: value TP_GND -> ~; footprint TestPoint:TestPoint_THTPad_D2.0mm_Drill1.0mm -> TestPoint:TestPoint_Loop_D2.50mm_Drill1.0mm; Comment (none) -> CM; DNP (none) -> DNP; Part (none) -> Keystone 5000
- U6: renamed from U8; footprint Package_TO_SOT_SMD:SOT-23-5_HandSoldering -> Package_TO_SOT_SMD:SOT-23-5
Connections:
- net labels added: +5V, BAL_CTRL1, BAL_CTRL2, BUCK_VCC, CAP_D1, CAP_D2, CAP_V0, CAP_V1, CAP_V2, CM, COMP, CS, CSG, DEMB, FB, GNDA, GNDPWR, HB, HO, IN_CS+, IN_CS-, I_SENSE, LO, RAMP, RT, SW, UVLO, VCAP1, VCAP2, V_CHARGE, V_IN
- net labels removed: +2V5, VIN_F, Vcap
- wire segments 74 -> 274
- no-connect marks 0 -> 2
Other:
- note added: "(need around 0.1 ohm ESR)"
- note added: "0.12V/A"
- note added: "0.6V/A"
- note added: "1.8-5.4V"
- note added: "100khz when light load\n400khz when heavy load"
- note added: "10V UVLO"
- note added: "3.6V"
- note added: "5.33V"
- note added: "5V aux supply\nfor power supply\nduring charge"
- note added: "Adaptive\nswitching\nfrequency"
- note added: "Buck-boost\nconverter"
- note added: "Buck\nconverter\nfor\ncharging"
- note added: "EMI Filter"
- note added: "Ideal diode"
- note added: "Input current limit\n5A"
- note added: "Layout notes:\n- Keep current loops short:\nInput Cap -> HS FET -> LS FET -> Sense R -> GND -> Input Cap (important)\nInductor -> Output Cap -> GND -> Sense R -> LS FET -> Inductor (less important)\n- Keep switching FETs close to controller\n- Consider thermals for switching FETs and balancing BJTs"
- note added: "Output current limit"
- note added: "Reverse\nBlocking\nMosfet"
- note added: "Supercapacitor\nbalancing"
- note added: "Supercapacitor\npower backup"
- note removed: "2.5-5.2V operating"
- note removed: "250kHz\nswitching\nfrequency"
- note removed: "5.2V output"
- note removed: "Current\nMeasure"
- note removed: "Discharge"
- note removed: "Energy\nStorage"
- note removed: "SCCU30B356SRB"
- note removed: "UVLO 10V"
- moved on the sheet: U6

Commit message: Main board; tweak feedback compensation network
Parts:
- C27: value 150pF -> 1nF
Other:
- note added: "Buck converter layout notes:\n- Keep current loops short:\nInput Cap -> HS FET -> LS FET -> Sense R -> GND -> Input Cap (important)\nInductor -> Output Cap -> GND -> Sense R -> LS FET -> Inductor (less important)\n- Keep switching FETs close to controller\n- Keep compensation network close to controller\n- Consider thermals for switching FETs and balancing BJTs"
- note removed: "Layout notes:\n- Keep current loops short:\nInput Cap -> HS FET -> LS FET -> Sense R -> GND -> Input Cap (important)\nInductor -> Output Cap -> GND -> Sense R -> LS FET -> Inductor (less important)\n- Keep switching FETs close to controller\n- Consider thermals for switching FETs and balancing BJTs"
Changed lines of the file:
@@
 P 1650 3900
 F 0 "C27" V 1600 3950 50  0000 L CNN
-F 1 "150pF" V 1600 3850 50  0000 R CNN
+F 1 "1nF" V 1600 3850 50  0000 R CNN
 F 2 "Capacitor_SMD:C_0402_1005Metric" H 1650 3900 50  0001 C CNN
 F 3 "~" H 1650 3900 50  0001 C CNN
@@
 Buck\nconverter\nfor\ncharging
 Text Notes 3500 6000 0    50   ~ 0
-Layout notes:\n- Keep current loops short:\nInput Cap -> HS FET -> LS FET -> Sense R -> GND -> Input Cap (important)\nInductor -> Output Cap -> GND -> Sense R -> LS FET -> Inductor (less important)\n- Keep switching FETs close to controller\n- Consider thermals for switching FETs and balancing BJTs
+Buck converter layout notes:\n- Keep current loops short:\nInput Cap -> HS FET -> LS FET -> Sense R -> GND -> Input Cap (important)\nInductor -> Output Cap -> GND -> Sense R -> LS FET -> Inductor (less important)\n- Keep switching FETs close to controller\n- Keep compensation network close to controller\n- Consider thermals for switching FETs and balancing BJTs
 Text Notes 6400 4050 0    50   ~ 0
 Supercapacitor\npower backup

Commit message: Main board: final change to compensation network
None of this really matters with the supercaps at the output,
just trying to optimize the loop without them.
Parts:
- C27: value 1nF -> 100pF
- C29: value 0.1uF -> 1nF
- R23: value 10k -> 47k
- R33, R38, R44: footprint Resistor_SMD:R_0805_2012Metric -> Resistor_SMD:R_0402_1005Metric
Changed lines of the file:
@@
 F 0 "R44" H 9991 5954 50  0000 R CNN
 F 1 "47k" H 9991 6045 50  0000 R CNN
-F 2 "Resistor_SMD:R_0805_2012Metric" H 10050 6000 50  0001 C CNN
+F 2 "Resistor_SMD:R_0402_1005Metric" H 10050 6000 50  0001 C CNN
 F 3 "~" H 10050 6000 50  0001 C CNN
 	1    10050 6000
@@
 F 0 "R38" H 9991 5354 50  0000 R CNN
 F 1 "47k" H 9991 5445 50  0000 R CNN
-F 2 "Resistor_SMD:R_0805_2012Metric" H 10050 5400 50  0001 C CNN
+F 2 "Resistor_SMD:R_0402_1005Metric" H 10050 5400 50  0001 C CNN
 F 3 "~" H 10050 5400 50  0001 C CNN
 	1    10050 5400
@@
 	1    9250 3700
 	1    0    0    -1
-$EndComp
-$Comp
-L Device:L L4
-U 1 1 602ECEC9
-P 4350 4100
-F 0 "L4" V 4540 4100 50  0000 C CNN
-F 1 "3.3uH" V 4449 4100 50  0000 C CNN
-F 2 "Inductor_SMD:L_Bourns_SRP1245A" H 4350 4100 50  0001 C CNN
-F 3 "~" H 4350 4100 50  0001 C CNN
-F 4 "SRP1265A-3R3M" V 4350 4100 50  0001 C CNN "Part"
-	1    4350 4100
-	0    -1   -1   0
 $EndComp
 $Comp
@@
 F 0 "R33" H 1592 4746 50  0000 R CNN
 F 1 "47k" H 1592 4655 50  0000 R CNN
-F 2 "Resistor_SMD:R_0805_2012Metric" H 1650 4700 50  0001 C CNN
+F 2 "Resistor_SMD:R_0402_1005Metric" H 1650 4700 50  0001 C CNN
 F 3 "~" H 1650 4700 50  0001 C CNN
 	1    1650 4700
@@
 P 1500 4100
 F 0 "R23" V 1550 4200 50  0000 L CNN
-F 1 "10k" V 1400 4100 50  0000 C CNN
+F 1 "47k" V 1400 4100 50  0000 C CNN
 F 2 "Resistor_SMD:R_0402_1005Metric" H 1500 4100 50  0001 C CNN
 F 3 "~" H 1500 4100 50  0001 C CNN
@@
 P 1800 4100
 F 0 "C29" V 1850 4150 50  0000 L CNN
-F 1 "0.1uF" V 1700 4100 50  0000 C CNN
+F 1 "1nF" V 1700 4100 50  0000 C CNN
 F 2 "Capacitor_SMD:C_0402_1005Metric" H 1800 4100 50  0001 C CNN
 F 3 "~" H 1800 4100 50  0001 C CNN
@@
 P 1650 3900
 F 0 "C27" V 1600 3950 50  0000 L CNN
-F 1 "1nF" V 1600 3850 50  0000 R CNN
+F 1 "100pF" V 1600 3850 50  0000 R CNN
 F 2 "Capacitor_SMD:C_0402_1005Metric" H 1650 3900 50  0001 C CNN
 F 3 "~" H 1650 3900 50  0001 C CNN
@@
 Wire Notes Line
 	3500 1950 6500 1950
+$Comp
+L Device:L L4
+U 1 1 602ECEC9
+P 4350 4100
+F 0 "L4" V 4540 4100 50  0000 C CNN
+F 1 "3.3uH" V 4449 4100 50  0000 C CNN
+F 2 "Inductor_SMD:L_Bourns_SRP1245A" H 4350 4100 50  0001 C CNN
+F 3 "~" H 4350 4100 50  0001 C CNN
+F 4 "SRP1265A-3R3M" V 4350 4100 50  0001 C CNN "Part"
+	1    4350 4100
+	0    -1   -1   0
+$EndComp
 $EndSCHEMATC

Commit message: Added first rev of design of new TSAL main board
Parts:
- C18, C19, C33, C34, C36, C37: symbol Device:C_Polarized_US -> TSAL-rescue:C_Polarized_US-Device
- D3: symbol Device:D_Schottky_Small_Filled -> TSAL-rescue:D_Schottky_Small_Filled-Device
- F1, F2: footprint Fuse:Fuseholder_Littelfuse_Nano2_154x -> footprints_archive_old_design:Fuseholder_Littelfuse_Nano2_154x
- L1: value 1uH -> 1.5uH; footprint Inductor_SMD:L_1206_3216Metric -> Inductor_SMD:L_Bourns-SRN4018; Part LB3218T1R0M -> SRN4018-1R5Y
- U8: symbol Device:Opamp_Quad -> TSAL-rescue:Opamp_Quad-Device
Changed lines of the file:
@@
 $EndComp
 $Comp
-L Device:Opamp_Quad U8
+L TSAL-rescue:Opamp_Quad-Device U8
 U 3 1 616C69E2
 P 9250 5400
@@
 $EndComp
 $Comp
-L Device:Opamp_Quad U8
+L TSAL-rescue:Opamp_Quad-Device U8
 U 4 1 616C7F69
 P 9250 6000
@@
 $EndComp
 $Comp
-L Device:Opamp_Quad U8
+L TSAL-rescue:Opamp_Quad-Device U8
 U 2 1 616C4A34
 P 9250 4700
@@
 $EndComp
 $Comp
-L Device:Opamp_Quad U8
+L TSAL-rescue:Opamp_Quad-Device U8
 U 1 1 615ADA58
 P 9250 3700
@@
 F 0 "F2" V 9763 1800 50  0000 C CNN
 F 1 "1A" V 9854 1800 50  0000 C CNN
-F 2 "Fuse:Fuseholder_Littelfuse_Nano2_154x" V 9980 1800 50  0001 C CNN
+F 2 "footprints_archive_old_design:Fuseholder_Littelfuse_Nano2_154x" V 9980 1800 50  0001 C CNN
 F 3 "~" H 10050 1800 50  0001 C CNN
 F 4 "154001.0" V 9945 1800 50  0000 C CNN "Part"
@@
 	1    3800 1650
 	1    0    0    -1
-$EndComp
-$Comp
-L Device:L L1
-U 1 1 603C095D
-P 8600 1450
-F 0 "L1" V 8790 1450 50  0000 C CNN
-F 1 "1uH" V 8699 1450 50  0000 C CNN
-F 2 "Inductor_SMD:L_1206_3216Metric" H 8600 1450 50  0001 C CNN
-F 3 "~" H 8600 1450 50  0001 C CNN
-F 4 "LB3218T1R0M" V 8600 1450 50  0001 C CNN "Part"
-	1    8600 1450
-	0    -1   -1   0
 $EndComp
 $Comp
@@
 $EndComp
 $Comp
-L Device:Opamp_Quad U8
+L TSAL-rescue:Opamp_Quad-Device U8
 U 5 1 616A1882
 P 6100 7000
@@
 F 0 "F1" V 963 1500 50  0000 C CNN
 F 1 "6A" V 1054 1500 50  0000 C CNN
-F 2 "Fuse:Fuseholder_Littelfuse_Nano2_154x" V 1180 1500 50  0001 C CNN
+F 2 "footprints_archive_old_design:Fuseholder_Littelfuse_Nano2_154x" V 1180 1500 50  0001 C CNN
 F 3 "~" H 1250 1500 50  0001 C CNN
 F 4 "15406.3" V 1145 1500 50  0000 C CNN "Part"
@@
 $EndComp
 $Comp
-L Device:D_Schottky_Small_Filled D3
+L TSAL-rescue:D_Schottky_Small_Filled-Device D3
 U 1 1 602CFF2F
 P 3250 3750
@@
 $EndComp
 $Comp
-L Device:C_Polarized_US C33
+L TSAL-rescue:C_Polarized_US-Device C33
 U 1 1 60398AFC
 P 6200 4400
+AR Path="/60398AFC" Ref="C33"  Part="1"
+AR Path="/5DE07D62/60398AFC" Ref="C33"  Part="1"
 F 0 "C33" H 6315 4446 50  0000 L CNN
 F 1 "200F" H 6315 4355 50  0000 L CNN
@@
 $EndComp
 $Comp
-L Device:C_Polarized_US C36
+L TSAL-rescue:C_Polarized_US-Device C36
 U 1 1 60399785
 P 6200 4800
+AR Path="/60399785" Ref="C36"  Part="1"
+AR Path="/5DE07D62/60399785" Ref="C36"  Part="1"
 F 0 "C36" H 6315 4846 50  0000 L CNN
 F 1 "200F" H 6315 4755 50  0000 L CNN
@@
 $EndComp
 $Comp
-L Device:C_Polarized_US C34
+L TSAL-rescue:C_Polarized_US-Device C34
 U 1 1 6039DE0A
 P 6700 4400
+AR Path="/6039DE0A" Ref="C34"  Part="1"
+AR Path="/5DE07D62/6039DE0A" Ref="C34"  Part="1"
 F 0 "C34" H 6815 4446 50  0000 L CNN
 F 1 "200F" H 6815 4355 50  0000 L CNN
@@
 $EndComp
 $Comp
-L Device:C_Polarized_US C37
+L TSAL-rescue:C_Polarized_US-Device C37
 U 1 1 6039DE10
 P 6700 4800
+AR Path="/6039DE10" Ref="C37"  Part="1"
+AR Path="/5DE07D62/6039DE10" Ref="C37"  Part="1"
 F 0 "C37" H 6815 4846 50  0000 L CNN
 F 1 "200F" H 6815 4755 50  0000 L CNN
@@
 $EndComp
 $Comp
-L Device:C_Polarized_US C18
+L TSAL-rescue:C_Polarized_US-Device C18
 U 1 1 604522CD
 P 2800 2550
+AR Path="/604522CD" Ref="C18"  Part="1"
+AR Path="/5DE07D62/604522CD" Ref="C18"  Part="1"
 F 0 "C18" H 2915 2596 50  0000 L CNN
 F 1 "220uF" H 2915 2505 50  0000 L CNN
@@
 $EndComp
 $Comp
-L Device:C_Polarized_US C19
+L TSAL-rescue:C_Polarized_US-Device C19
 U 1 1 6136B917
 P 3500 2550
+AR Path="/6136B917" Ref="C19"  Part="1"
+AR Path="/5DE07D62/6136B917" Ref="C19"  Part="1"
 F 0 "C19" H 3615 2596 50  0000 L CNN
 F 1 "220uF" H 3615 2505 50  0000 L CNN
@@
 	0    -1   -1   0
 $EndComp
+$Comp
+L Device:L L1
+U 1 1 603C095D
+P 8600 1450
+F 0 "L1" V 8790 1450 50  0000 C CNN
+F 1 "1.5uH" V 8699 1450 50  0000 C CNN
+F 2 "Inductor_SMD:L_Bourns-SRN4018" H 8600 1450 50  0001 C CNN
+F 3 "~" H 8600 1450 50  0001 C CNN
+F 4 "SRN4018-1R5Y" V 8600 1450 50  0001 C CNN "Part"
+	1    8600 1450
+	0    -1   -1   0
+$EndComp
