File: Main/TSAL.kicad_pcb (KiCad board)
At the start: 2 copper layers, 140 x 70 mm, 156 parts, among them J1 Micro-Fit, J2 Mini-SPOX, J3 Mini-SPOX, J4 Mini-SPOX, J5 Mini-SPOX, Q1 IRLML2502, Q10 NPN, Q11 MJD122, Q12 PNP, Q2 IRLML2502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

Commit message: hv sense v2
Other:
- net class Default removed
